Commit message: ur3 and door appear before fixing collisions

File: assets/urdf/door_test/ur3.urdf (robot description, URDF)
Before this commit: robot ur3_robot, 11 links, 10 joints
Joints:
- joint base_link-base_link_inertia: origin xyz=0 0 0 rpy=0 0 3.141592653589793 -> xyz=0 0 0.8 rpy=0 0 -4.712389
