Commit message: minor change

File: assets/urdf/door_test/hook_test copy.urdf (robot description, URDF)
Before this commit: robot hook_test, 10 links, 9 joints
Links:
- link hook: geometry collision mesh filename=./meshes/ur3/collision/hook4door_2_asm.obj scale=0.001 0.001 0.001; visual mesh filename=./meshes/ur3/collision/hook4door_2_asm.obj scale=0.001 0.001 0.001
Joints:
- joint ee_rx: limit lower=-0.1 upper=0.1 effort=100.0 velocity=1.0 -> lower=-0.1 upper=0.1 effort=10000.0 velocity=1.0
- joint ee_ry: limit lower=-0.1 upper=0.1 effort=100.0 velocity=1.0 -> lower=-0.1 upper=0.1 effort=10000.0 velocity=1.0
- joint ee_rz: limit lower=-0.1 upper=0.1 effort=100.0 velocity=1.0 -> lower=-0.1 upper=0.1 effort=10000.0 velocity=1.0
- joint ee_x: limit lower=-0.5 upper=0.5 effort=100.0 velocity=1.0 -> lower=-0.5 upper=0.5 effort=10000.0 velocity=1.0
- joint ee_y: limit lower=-0.5 upper=0.5 effort=100.0 velocity=1.0 -> lower=-0.1 upper=0.1 effort=10000.0 velocity=1.0
- joint ee_z: limit lower=-0.5 upper=0.5 effort=100.0 velocity=1.0 -> lower=-0.4 upper=0.4 effort=10000.0 velocity=1.0
