Commit message: add left door(in progress) and enhance door damping fuctor

File: assets/urdf/door_test/door_2.urdf (robot description, URDF)
Before this commit: robot door_test, 5 links, 4 joints
Joints:
- joint base_joint: origin xyz=0 0.5 0.0 rpy=0 0 3.14 -> xyz=0 0.5 0.0 rpy=0 0 0

Commit message: add left hinge door : door_2.urdf

File: assets/urdf/door_test/door_2.urdf (robot description, URDF)
Before this commit: robot door_test, 5 links, 4 joints
Joints:
- joint door_handle: axis 1 0 0 -> -1 0 0
- joint door_hinge: origin xyz=0.432 0.06858 2.040 -> xyz=0.525 0.06858 0 rpy=0 3.14159 0
