Commit message: minor change

File: assets/urdf/door_test/door_1.urdf (robot description, URDF)
Before this commit: robot door_1, 4 links, 3 joints
Links:
- added link world
- link door_frame: mass 1000.0 -> 10000.0; geometry collision box size=0.05029 0.06858 2.10820; collision box size=0.05029 0.06858 2.10820
Joints:
- added joint world2base: type fixed, parent world, child base_link

Commit message: ur3 moved! but door bug not fixed

File: assets/urdf/door_test/door_1.urdf (robot description, URDF)
Before this commit: robot door_test, 5 links, 4 joints
Links:
- link door: geometry collision mesh filename=./meshes/door.dae; visual mesh filename=./meshes/door.dae
- link door_frame: geometry collision box size=0.05029 0.06858 2.10820; collision box size=0.05029 0.06858 2.10820
- link door_handles: geometry collision mesh filename=./meshes/door_handle.dae; visual mesh filename=./meshes/door_handle.dae

File: assets/urdf/door_test/ur3.urdf (robot description, URDF)
Before this commit: robot ur3_robot, 11 links, 10 joints
Links:
- link base_link_inertia: geometry collision mesh filename=./meshes/ur3/collision/base.stl; visual mesh filename=./meshes/ur3/visual/base.dae
- link forearm_link: geometry collision mesh filename=./meshes/ur3/collision/forearm.stl; visual mesh filename=./meshes/ur3/visual/forearm.dae
- link shoulder_link: geometry collision mesh filename=./meshes/ur3/collision/shoulder.stl; visual mesh filename=./meshes/ur3/visual/shoulder.dae
- link upper_arm_link: geometry collision mesh filename=./meshes/ur3/collision/upperarm.stl; visual mesh filename=./meshes/ur3/visual/upperarm.dae
- link wrist_1_link: geometry collision mesh filename=./meshes/ur3/collision/wrist1.stl; visual mesh filename=./meshes/ur3/visual/wrist1.dae
- link wrist_2_link: geometry collision mesh filename=./meshes/ur3/collision/wrist2.stl; visual mesh filename=./meshes/ur3/visual/wrist2.dae
- link wrist_3_link: geometry collision mesh filename=./meshes/ur3/collision/wrist3.stl; visual mesh filename=./meshes/ur3/visual/wrist3.dae

Commit message: minor change of door

File: assets/urdf/door_test/door_1.urdf (robot description, URDF)
Before this commit: robot door_test, 5 links, 4 joints
Links:
- removed link world
Joints:
- removed joint world2base

File: assets/urdf/sektion_cabinet_model/urdf/sektion_cabinet.urdf (robot description, URDF)
Before this commit: robot cabinet_sektion, 9 links, 8 joints
Links:
- added link world
Joints:
- added joint world_to_sektion: type fixed, parent world, child sektion, origin xyz=0.85 0 0.38 rpy=0 0 3.14159

Commit message: ur3 self collisions solved

File: assets/urdf/door_test/door_1.urdf (robot description, URDF)
Before this commit: robot door_test, 4 links, 3 joints
Joints:
- joint base_joint: origin xyz=0.4 -0.5 -0.4 -> xyz=0.0 -0.5 -0.4
- joint door_handle: axis (none) -> 1 0 0; origin xyz=0.013 0.8 -1.0 -> xyz=0.013 0.75 -1.0
- joint door_hinge: origin xyz=-0.06 0.06858 2.040 -> xyz=0.432 0.06858 2.040

File: assets/urdf/door_test/ur3_hand.urdf (robot description, URDF)
Before this commit: robot ur3_robot, 11 links, 10 joints
Links:
- removed link tool0
- added link hand_base; collision mesh filename=./meshes/ur3/collision/hand_base.obj; visual mesh filename=./meshes/ur3/visual/hand_base.dae
- added link hand_left; collision mesh filename=./meshes/ur3/collision/finger.obj; visual mesh filename=./meshes/ur3/visual/finger.dae
- added link hand_right; collision mesh filename=./meshes/ur3/collision/finger.obj; visual mesh filename=./meshes/ur3/visual/finger.dae
- link base_link_inertia: geometry collision mesh filename=./meshes/ur3/collision/base.obj; visual mesh filename=./meshes/ur3/visual/base.dae
- link forearm_link: geometry collision mesh filename=./meshes/ur3/collision/forearm.obj; visual mesh filename=./meshes/ur3/visual/forearm.dae
- link shoulder_link: geometry collision mesh filename=./meshes/ur3/collision/shoulder.obj; visual mesh filename=./meshes/ur3/visual/shoulder.dae
- link upper_arm_link: geometry collision mesh filename=./meshes/ur3/collision/upperarm.obj; visual mesh filename=./meshes/ur3/visual/upperarm.dae
- link wrist_1_link: geometry collision mesh filename=./meshes/ur3/collision/wrist1.obj; visual mesh filename=./meshes/ur3/visual/wrist1.dae
- link wrist_2_link: geometry collision mesh filename=./meshes/ur3/collision/wrist2.obj; visual mesh filename=./meshes/ur3/visual/wrist2.dae
- link wrist_3_link: geometry collision mesh filename=./meshes/ur3/collision/wrist3.obj; visual mesh filename=./meshes/ur3/visual/wrist3.dae
Joints:
- removed joint flange-tool0
- added joint ur3_handjoint: type fixed, parent flange, child hand_base, origin xyz=0.05 0 0 rpy=1.5707963267948966 0 1.5707963267948966
- added joint ur3_lefthandjoint: type prismatic, parent hand_base, child hand_left, origin xyz=-0.016 0 0.075 rpy=0 0 -1.5707963267948966, axis 0 1 0, limit lower=0 upper=0.016 effort=1000 velocity=0.1
- added joint ur3_righthandjoint: type prismatic, parent hand_base, child hand_right, origin xyz=0.016 0 0.075 rpy=0 0 1.5707963267948966, axis 0 1 0, limit lower=0 upper=0.016 effort=1000.0 velocity=0.1
- joint shoulder_lift_joint: origin xyz=0 0 0 rpy=1.570796327 0 0 -> xyz=0 0 0 rpy=1.570796327 1.570796327 0
- joint wrist_1_joint: origin xyz=-0.21325 0 0.11235 rpy=0 0 0 -> xyz=-0.21325 0 0.11235 rpy=0 0 -1.570796327

File: assets/urdf/franka_description/robots/franka_panda.urdf (robot description, URDF)
Before this commit: robot panda, 11 links, 10 joints
Links:
- link panda_link5: geometry collision mesh filename=package://franka_description/meshes/collision/link5.obj scale=1.0 1.0 1.0; visual mesh filename=package://franka_description/meshes/visual/link5.dae

Commit message: m

File: assets/urdf/door_test/door_1.urdf (robot description, URDF)
Before this commit: robot door_test, 4 links, 3 joints
Links:
- link door_handles: geometry collision mesh filename=./meshes/door_handle.dae; collision mesh filename=./meshes/door_handle.dae
Joints:
- joint base_joint: origin xyz=0.0 -0.5 -0.4 -> xyz=0.0 -0.5 -0.4 rpy=0 0 3.14

File: assets/urdf/door_test/hook_test.urdf (robot description, URDF)
Before this commit: robot hook_test, 10 links, 9 joints
Joints:
- joint hand2hook: origin xyz=0 0 0 rpy=1.57 0 3.14159 -> xyz=0.03 0 0.03 rpy=1.57 0 3.14159

Commit message: minor change to read tensors

File: assets/urdf/door_test/door_1.urdf (robot description, URDF)
Before this commit: robot door_test, 4 links, 3 joints
Joints:
- joint base_joint: origin xyz=0.0 -0.5 -0.4 rpy=0 0 3.14 -> xyz=0 0.5 -0.4 rpy=0 0 3.14

Commit message: defined d_imgs and start to make obsefvation space

File: assets/urdf/door_test/door_1.urdf (robot description, URDF)
Before this commit: robot door_test, 4 links, 3 joints
Joints:
- joint base_joint: origin xyz=0 0.5 -0.4 rpy=0 0 3.14 -> xyz=0 0.5 0.0 rpy=0 0 3.14

File: assets/urdf/door_test/hook_test.urdf (robot description, URDF)
Before this commit: robot hook_test, 10 links, 9 joints
Joints:
- joint baselink2eebase: origin xyz=0 0 0.5 rpy=0 0 0 -> xyz=0 0 0 rpy=0 0 0

Commit message: minor change

File: assets/urdf/door_test/door_1.urdf (robot description, URDF)
Before this commit: robot door_test, 4 links, 3 joints
Joints:
- joint door_handle: limit lower=0 upper=0.785 effort=100 velocity=1000.00 -> lower=0 upper=0.5236 effort=100 velocity=1000.00

Commit message: change door friction, damping and handle position

File: assets/urdf/door_test/door_1.urdf (robot description, URDF)
Before this commit: robot door_test, 4 links, 3 joints
Joints:
- joint door_handle: origin xyz=0.013 0.75 -1.0 -> xyz=0.035 0.75 -1.0

Commit message: minor change

File: assets/urdf/door_test/door_1.urdf (robot description, URDF)
Before this commit: robot door_test, 4 links, 3 joints
Joints:
- joint door_hinge: limit lower=0 upper=1.57 effort=100 velocity=1000.00 -> lower=0 upper=1.57 effort=100 velocity=100.00

File: assets/urdf/door_test/hook_test.urdf (robot description, URDF)
Before this commit: robot hook_test, 10 links, 9 joints
Joints:
- joint ee_rx: limit lower=-0.1 upper=0.1 effort=10000.0 velocity=0.2 -> lower=-0.1 upper=0.1 effort=10000.0 velocity=1.0
- joint ee_ry: limit lower=-0.1 upper=0.1 effort=10000.0 velocity=0.2 -> lower=-0.1 upper=0.1 effort=10000.0 velocity=1.0
- joint ee_rz: limit lower=-0.1 upper=0.1 effort=10000.0 velocity=0.2 -> lower=-0.1 upper=0.1 effort=10000.0 velocity=1.0
- joint ee_x: limit lower=-0.5 upper=0.5 effort=10000.0 velocity=0.2 -> lower=-0.5 upper=0.5 effort=10000.0 velocity=1.0
- joint ee_y: limit lower=-0.1 upper=0.1 effort=10000.0 velocity=0.2 -> lower=-0.1 upper=0.1 effort=10000.0 velocity=1.0
- joint ee_z: limit lower=-0.4 upper=0.2 effort=10000.0 velocity=0.2 -> lower=-0.4 upper=0.4 effort=10000.0 velocity=1.0

Commit message: minor change

File: assets/urdf/door_test/door_1.urdf (robot description, URDF)
Before this commit: robot door_test, 4 links, 3 joints
Links:
- added link door_latch; collision box size=0.001 0.14 0.01
Joints:
- added joint handle2latch: type fixed, parent door_handles, child door_latch

File: assets/urdf/door_test/door_backup.urdf (robot description, URDF)
Before this commit: robot door_test, 4 links, 3 joints
Links:
- link door_handles: geometry collision mesh filename=./meshes/door_handle.dae; collision mesh filename=./meshes/door_handle.dae
Joints:
- joint base_joint: origin xyz=0.4 -0.5 -0.4 -> xyz=0 0.5 0.0 rpy=0 0 3.14
- joint door_handle: axis (none) -> 1 0 0; limit lower=0 upper=0.785 effort=100 velocity=1000.00 -> lower=0 upper=0.5236 effort=100 velocity=1000.00; origin xyz=0.013 0.8 -1.0 -> xyz=0.035 0.75 -1.0
- joint door_hinge: limit lower=0 upper=1.57 effort=100 velocity=1000.00 -> lower=0 upper=1.57 effort=100 velocity=100.00; origin xyz=-0.06 0.06858 2.040 -> xyz=0.432 0.06858 2.040

Commit message: edit door conditions

File: assets/urdf/door_test/door_1.urdf (robot description, URDF)
Before this commit: robot door_test, 5 links, 4 joints
Joints:
- joint door_hinge: limit lower=0 upper=1.57 effort=100 velocity=100.00 -> lower=0 upper=1.57 effort=10000 velocity=100.00

Commit message: large changes comes

File: assets/urdf/door_test/door_1.urdf (robot description, URDF)
Before this commit: robot door_test, 5 links, 4 joints
Joints:
- joint base_joint: origin xyz=0 0.5 0.0 rpy=0 0 3.14 -> xyz=0 0.6 0.0 rpy=0 0 3.14

File: assets/urdf/door_test/hook_test.urdf (robot description, URDF)
Before this commit: robot hook_test, 11 links, 10 joints
Joints:
- joint ee_rx: limit lower=-0.1 upper=0.1 effort=10.0 velocity=2.0 -> lower=-1.0 upper=1.0 effort=10.0 velocity=2.0
- joint ee_ry: limit lower=-0.1 upper=0.1 effort=10.0 velocity=2.0 -> lower=-1.0 upper=1.0 effort=10.0 velocity=2.0
- joint ee_rz: limit lower=-0.1 upper=0.1 effort=10.0 velocity=2.0 -> lower=-1.0 upper=1.0 effort=10.0 velocity=2.0
- joint ee_x: limit lower=-0.5 upper=1.0 effort=100.0 velocity=2.0 -> lower=-1.0 upper=1.0 effort=100.0 velocity=2.0
- joint ee_y: limit lower=-0.2 upper=0.2 effort=100.0 velocity=2.0 -> lower=-1.0 upper=1.0 effort=100.0 velocity=2.0
- joint ee_z: limit lower=-0.3 upper=0.3 effort=100.0 velocity=2.0 -> lower=-1.0 upper=1.0 effort=100.0 velocity=2.0

Commit message: while big minor change

File: assets/urdf/door_test/door_1.urdf (robot description, URDF)
Before this commit: robot door_test, 5 links, 4 joints
Joints:
- joint base_joint: origin xyz=0 0.6 0.0 rpy=0 0 3.14 -> xyz=0 0.0 0.0 rpy=0 0 3.14
- joint door_hinge: origin xyz=0.432 0.06858 2.040 -> xyz=-0.068 0.06858 2.040

File: assets/urdf/door_test/hook_test.urdf (robot description, URDF)
Before this commit: robot hook_test, 11 links, 10 joints
Joints:
- joint hand2hook: origin xyz=-0.029 0.031 0.045 rpy=-1.57 0 -1.57 -> xyz=-0.031 0.031 0.0425 rpy=-1.57 0 -1.57

Commit message: add ur3_dof_pos_prev

File: assets/urdf/door_test/door_1.urdf (robot description, URDF)
Before this commit: robot door_test, 5 links, 4 joints
Joints:
- joint base_joint: origin xyz=0 0.0 0.0 rpy=0 0 3.14 -> xyz=0 0.5 0.0 rpy=0 0 3.14
- joint door_hinge: origin xyz=-0.068 0.06858 2.040 -> xyz=-0.076 0.06858 2.040

Commit message: uni started reaching test

File: assets/urdf/door_test/door_1.urdf (robot description, URDF)
Before this commit: robot door_test, 5 links, 4 joints
Joints:
- joint door_handle: origin xyz=0.035 0.75 -1.0 -> xyz=0.035 0.75 -1.02

Commit message: door hinge bug fixed

File: assets/urdf/door_test/door_1.urdf (robot description, URDF)
Before this commit: robot door_test, 5 links, 4 joints
Joints:
- joint door_hinge: origin xyz=-0.076 0.06858 2.040 -> xyz=-0.07 0.06858 2.040
