Commit message: add inverse doors

File: assets/urdf/door_test/door_1_inv.urdf (robot description, URDF)
Before this commit: robot door_test, 5 links, 4 joints
Joints:
- joint base_joint: origin xyz=0 0.5 0.0 rpy=0 0 3.14159 -> xyz=0 0.5 0.0 rpy=0 0 0
- joint door_handle: axis 1 0 0 -> -1 0 0
- joint door_hinge: origin xyz=-0.07 0.06858 2.040 -> xyz=-0.07 0.972 0 rpy=3.14159 0 0

File: assets/urdf/door_test/door_2_inv.urdf (robot description, URDF)
Before this commit: robot door_test, 5 links, 4 joints
Joints:
- joint base_joint: origin xyz=0 0.5 0.0 rpy=0 0 3.14159 -> xyz=0 -0.5 0.0 rpy=0 0 0

Commit message: add all doors

File: assets/urdf/door_test/door_1_inv.urdf (robot description, URDF)
Before this commit: robot door_test, 5 links, 4 joints
Joints:
- joint base_joint: origin xyz=0 0.5 0.0 rpy=0 0 0 -> xyz=0 -0.5 0.0 rpy=0 0 0
