Commit message: added manipulator but, crasy jabobian

File: assets/urdf/door_test/ur3_hook.urdf (robot description, URDF)
Before this commit: robot ur3_robot, 11 links, 10 joints
Links:
- added link ee_rz_link
- added link hand_base; collision cylinder length=0.065 radius=0.033; visual cylinder length=0.065 radius=0.033
- added link hook; collision mesh filename=./meshes/ur3/visual/hook4door_v3.obj; visual mesh filename=./meshes/ur3/collision/hook4door_v3.obj
- added link hook_finger; visual sphere radius=0.007
Joints:
- added joint ee2hand_joint: type fixed, parent ee_rz_link, child hand_base, origin xyz=0 0 0 rpy=0 1.57 0
- added joint ee_rz: type fixed, parent tool0, child ee_rz_link, origin xyz=0 0 0 rpy=0 0 0
- added joint hand2hook: type fixed, parent hand_base, child hook, origin xyz=-0.031 0.031 0.0425 rpy=-1.57 0 -1.57
- added joint hook_finger: type fixed, parent hand_base, child hook_finger, origin xyz=0.08 0 0.17 rpy=0 0 0
- joint flange-tool0: origin xyz=0 0 0 rpy=1.5707963267948966 0 1.5707963267948966 -> xyz=0 0 0 rpy=-3.141592653589793 0 0

Commit message: add UR3 and Panda

File: assets/urdf/door_test/ur3_hook.urdf (robot description, URDF)
Before this commit: robot ur3_robot, 15 links, 14 joints
Joints:
- joint base_link-base_fixed_joint: origin xyz=0 0 0 rpy=0 0 3.141592653589793 -> (none)
- joint base_link-base_link_inertia: origin xyz=0 0 0 rpy=0 0 -4.712389 -> (none)
