Commit message: door_hook bug

File: assets/urdf/door_test/hook_test.urdf (robot description, URDF)
Before this commit: robot hook_test, 3 links, 7 joints
Links:
- link hook: geometry collision mesh filename=./meshes/ur3/collision/hook4door.obj; visual mesh filename=./meshes/ur3/collision/hook4door.obj

Commit message: 1206 done

File: assets/urdf/door_test/hook_test.urdf (robot description, URDF)
Before this commit: robot hook_test, 4 links, 7 joints
Links:
- added link empty_link_1
- added link empty_link_2
- added link empty_link_3
- added link empty_link_4
- added link empty_link_5
Joints:
- joint ee_x: axis 1 0 0 -> (none)

Commit message: complete hook urdf

File: assets/urdf/door_test/hook_test.urdf (robot description, URDF)
Before this commit: robot hook_test, 9 links, 7 joints
Links:
- removed link empty_link_1
- removed link empty_link_2
- removed link empty_link_3
- removed link empty_link_4
- removed link empty_link_5
- added link ee_rx_link
- added link ee_ry_link
- added link ee_rz_link
- added link ee_x_link
- added link ee_y_link
- added link ee_z_link
Joints:
- added joint baselink2eebase: type fixed, parent base_link, child ee_base, origin xyz=0 0 0.5 rpy=0 0 0
- added joint ee2hand_joint: type fixed, parent ee_rz_link, child hand_base, origin xyz=0 0 0 rpy=0 1.57 0
- joint ee_rx: child hand_base -> ee_rx_link; limit lower=-0.5 upper=0.5 effort=1000.0 velocity=0.1 -> lower=-0.1 upper=0.1 effort=500.0 velocity=0.1; parent ee_base -> ee_z_link
- joint ee_ry: child hand_base -> ee_ry_link; limit lower=-0.5 upper=0.5 effort=1000.0 velocity=0.1 -> lower=-0.1 upper=0.1 effort=500.0 velocity=0.1; parent ee_base -> ee_rx_link
- joint ee_rz: child hand_base -> ee_rz_link; limit lower=-0.5 upper=0.5 effort=1000.0 velocity=0.1 -> lower=-0.1 upper=0.1 effort=500.0 velocity=0.1; parent ee_base -> ee_ry_link
- joint ee_x: axis (none) -> 1 0 0; child hand_base -> ee_x_link; limit lower=-0.5 upper=0.5 effort=1000.0 velocity=0.1 -> lower=-1 upper=1 effort=500.0 velocity=0.1
- joint ee_y: child hand_base -> ee_y_link; limit lower=-0.5 upper=0.5 effort=1000.0 velocity=0.1 -> lower=-1 upper=1 effort=500.0 velocity=0.1; parent ee_base -> ee_x_link
- joint ee_z: child hand_base -> ee_z_link; limit lower=-0.5 upper=0.5 effort=1000.0 velocity=0.1 -> lower=-1 upper=1 effort=500.0 velocity=0.1; parent ee_base -> ee_y_link
- joint hand2hook: origin xyz=0 0 0 rpy=0 0 0 -> xyz=0 0 0 rpy=1.57 0 3.14159

Commit message: newhook hook4door2 integrated and works

File: assets/urdf/door_test/hook_test.urdf (robot description, URDF)
Before this commit: robot hook_test, 10 links, 9 joints
Links:
- link hand_base: geometry collision cylinder length=0.065 radius=0.0365; visual cylinder length=0.065 radius=0.0365
- link hook: geometry collision mesh filename=./meshes/ur3/collision/hook4door_2_asm.obj scale=0.001 0.001 0.001; visual mesh filename=./meshes/ur3/collision/hook4door_2_asm.obj scale=0.001 0.001 0.001
Joints:
- joint ee_x: limit lower=-1 upper=1 effort=500.0 velocity=0.1 -> lower=-0.1 upper=0.1 effort=500.0 velocity=0.1
- joint ee_y: limit lower=-1 upper=1 effort=500.0 velocity=0.1 -> lower=-0.1 upper=0.1 effort=500.0 velocity=0.1
- joint ee_z: limit lower=-1 upper=1 effort=500.0 velocity=0.1 -> lower=-0.1 upper=0.1 effort=500.0 velocity=0.1
- joint hand2hook: origin xyz=0.03 0 0.03 rpy=1.57 0 3.14159 -> xyz=-0.028 0.032 0.045 rpy=-1.57 0 -1.57

Commit message: add cameras does work!!!!!!!!!!!!!

File: assets/urdf/door_test/hook_test.urdf (robot description, URDF)
Before this commit: robot hook_test, 10 links, 9 joints
Links:
- link hand_base: geometry collision cylinder length=0.065 radius=0.031; visual cylinder length=0.065 radius=0.031
Joints:
- joint ee_rx: limit lower=-0.1 upper=0.1 effort=500.0 velocity=0.1 -> lower=-10 upper=10 effort=500.0 velocity=10
- joint ee_ry: limit lower=-0.1 upper=0.1 effort=500.0 velocity=0.1 -> lower=-10 upper=10 effort=500.0 velocity=10
- joint ee_rz: limit lower=-0.1 upper=0.1 effort=500.0 velocity=0.1 -> lower=-10 upper=10 effort=500.0 velocity=10
- joint ee_x: limit lower=-0.1 upper=0.1 effort=500.0 velocity=0.1 -> lower=-10 upper=10 effort=500.0 velocity=10
- joint ee_y: limit lower=-0.1 upper=0.1 effort=500.0 velocity=0.1 -> lower=-10 upper=10 effort=500.0 velocity=10
- joint ee_z: limit lower=-0.1 upper=0.1 effort=500.0 velocity=0.1 -> lower=-10 upper=10 effort=500.0 velocity=10
- joint hand2hook: origin xyz=-0.028 0.032 0.045 rpy=-1.57 0 -1.57 -> xyz=-0.029 0.031 0.045 rpy=-1.57 0 -1.57

Commit message: camera position defined

File: assets/urdf/door_test/hook_test.urdf (robot description, URDF)
Before this commit: robot hook_test, 10 links, 9 joints
Joints:
- joint ee_rx: limit lower=-10 upper=10 effort=500.0 velocity=10 -> lower=-1 upper=1 effort=500.0 velocity=1
- joint ee_ry: limit lower=-10 upper=10 effort=500.0 velocity=10 -> lower=-1 upper=1 effort=500.0 velocity=1
- joint ee_rz: limit lower=-10 upper=10 effort=500.0 velocity=10 -> lower=-1 upper=1 effort=500.0 velocity=1
- joint ee_x: limit lower=-10 upper=10 effort=500.0 velocity=10 -> lower=-1 upper=1 effort=500.0 velocity=1
- joint ee_y: limit lower=-10 upper=10 effort=500.0 velocity=10 -> lower=-1 upper=1 effort=500.0 velocity=1
- joint ee_z: limit lower=-10 upper=10 effort=500.0 velocity=10 -> lower=-1 upper=1 effort=500.0 velocity=1

Commit message: action defined bad reward

File: assets/urdf/door_test/hook_test.urdf (robot description, URDF)
Before this commit: robot hook_test, 10 links, 9 joints
Joints:
- joint ee_rx: limit lower=-1 upper=1 effort=500.0 velocity=1 -> lower=-1 upper=1 effort=10000.0 velocity=1
- joint ee_ry: limit lower=-1 upper=1 effort=500.0 velocity=1 -> lower=-1 upper=1 effort=10000.0 velocity=1
- joint ee_rz: limit lower=-1 upper=1 effort=500.0 velocity=1 -> lower=-1 upper=1 effort=10000.0 velocity=1
- joint ee_x: limit lower=-1 upper=1 effort=500.0 velocity=1 -> lower=-0.3 upper=0.3 effort=10000.0 velocity=0.2
- joint ee_y: limit lower=-1 upper=1 effort=500.0 velocity=1 -> lower=-0.3 upper=0.3 effort=10000.0 velocity=0.2
- joint ee_z: limit lower=-1 upper=1 effort=500.0 velocity=1 -> lower=-0.3 upper=0.3 effort=10000.0 velocity=0.2

Commit message: minor change

File: assets/urdf/door_test/hook_test.urdf (robot description, URDF)
Before this commit: robot hook_test, 10 links, 9 joints
Joints:
- joint ee_x: limit lower=-0.3 upper=0.3 effort=10000.0 velocity=0.2 -> lower=-0.5 upper=0.5 effort=10000.0 velocity=0.2
- joint ee_y: limit lower=-0.3 upper=0.3 effort=10000.0 velocity=0.2 -> lower=-0.5 upper=0.5 effort=10000.0 velocity=0.2
- joint ee_z: limit lower=-0.3 upper=0.3 effort=10000.0 velocity=0.2 -> lower=-0.5 upper=0.5 effort=10000.0 velocity=0.2

Commit message: 1218 done

File: assets/urdf/door_test/hook_test.urdf (robot description, URDF)
Before this commit: robot hook_test, 10 links, 9 joints
Joints:
- joint ee_rx: limit lower=-1 upper=1 effort=10000.0 velocity=1 -> lower=-0.5 upper=0.5 effort=10000.0 velocity=0.2
- joint ee_ry: limit lower=-1 upper=1 effort=10000.0 velocity=1 -> lower=-0.5 upper=0.5 effort=10000.0 velocity=0.2
- joint ee_rz: limit lower=-1 upper=1 effort=10000.0 velocity=1 -> lower=-0.5 upper=0.5 effort=10000.0 velocity=0.2

Commit message: add handle reward, edit y limit on urdf, add action penalty and SAC modules(this doesnt work

File: assets/urdf/door_test/hook_test.urdf (robot description, URDF)
Before this commit: robot hook_test, 10 links, 9 joints
Joints:
- joint ee_y: limit lower=-0.5 upper=0.5 effort=10000.0 velocity=0.2 -> lower=-0.1 upper=0.1 effort=10000.0 velocity=0.2

Commit message: 1220 while learning, reduced damping, d_img normalized

File: assets/urdf/door_test/hook_test.urdf (robot description, URDF)
Before this commit: robot hook_test, 10 links, 9 joints
Joints:
- joint ee_z: limit lower=-0.5 upper=0.5 effort=10000.0 velocity=0.2 -> lower=-0.4 upper=0.2 effort=10000.0 velocity=0.2

Commit message: 1220 done, but wasnt better

File: assets/urdf/door_test/hook_test.urdf (robot description, URDF)
Before this commit: robot hook_test, 10 links, 9 joints
Joints:
- joint ee_rx: limit lower=-0.5 upper=0.5 effort=10000.0 velocity=0.2 -> lower=-0.1 upper=0.1 effort=10000.0 velocity=0.2
- joint ee_ry: limit lower=-0.5 upper=0.5 effort=10000.0 velocity=0.2 -> lower=-0.1 upper=0.1 effort=10000.0 velocity=0.2
- joint ee_rz: limit lower=-0.5 upper=0.5 effort=10000.0 velocity=0.2 -> lower=-0.1 upper=0.1 effort=10000.0 velocity=0.2

Commit message: before change network

File: assets/urdf/door_test/hook_test.urdf (robot description, URDF)
Before this commit: robot hook_test, 10 links, 9 joints
Joints:
- joint ee_rx: limit lower=-0.1 upper=0.1 effort=100.0 velocity=1.0 -> lower=-0.1 upper=0.1 effort=1000.0 velocity=1.0
- joint ee_ry: limit lower=-0.1 upper=0.1 effort=100.0 velocity=1.0 -> lower=-0.1 upper=0.1 effort=1000.0 velocity=1.0
- joint ee_rz: limit lower=-0.1 upper=0.1 effort=100.0 velocity=1.0 -> lower=-0.1 upper=0.1 effort=1000.0 velocity=1.0
- joint ee_x: limit lower=-0.5 upper=0.5 effort=100.0 velocity=1.0 -> lower=-0.5 upper=0.5 effort=1000.0 velocity=1.0
- joint ee_y: limit lower=-0.5 upper=0.5 effort=100.0 velocity=1.0 -> lower=-0.1 upper=0.1 effort=1000.0 velocity=1.0
- joint ee_z: limit lower=-0.5 upper=0.5 effort=100.0 velocity=1.0 -> lower=-0.4 upper=0.4 effort=1000.0 velocity=1.0

Commit message: 1221 done before distance reward

File: assets/urdf/door_test/hook_test.urdf (robot description, URDF)
Before this commit: robot hook_test, 10 links, 9 joints
Joints:
- joint ee_rx: limit lower=-0.1 upper=0.1 effort=1000.0 velocity=1.0 -> lower=-0.1 upper=0.1 effort=10.0 velocity=2.0
- joint ee_ry: limit lower=-0.1 upper=0.1 effort=1000.0 velocity=1.0 -> lower=-0.1 upper=0.1 effort=10.0 velocity=2.0
- joint ee_rz: limit lower=-0.1 upper=0.1 effort=1000.0 velocity=1.0 -> lower=-0.1 upper=0.1 effort=10.0 velocity=2.0
- joint ee_x: limit lower=-0.5 upper=0.5 effort=1000.0 velocity=1.0 -> lower=-0.5 upper=0.5 effort=10.0 velocity=2.0
- joint ee_y: limit lower=-0.1 upper=0.1 effort=1000.0 velocity=1.0 -> lower=-0.2 upper=0.2 effort=10.0 velocity=2.0
- joint ee_z: limit lower=-0.4 upper=0.4 effort=1000.0 velocity=1.0 -> lower=-0.3 upper=0.3 effort=10.0 velocity=2.0

Commit message: added dist reward and no clamp

File: assets/urdf/door_test/hook_test.urdf (robot description, URDF)
Before this commit: robot hook_test, 10 links, 9 joints
Joints:
- joint ee_x: limit lower=-0.5 upper=0.5 effort=10.0 velocity=2.0 -> lower=-0.5 upper=1.0 effort=10.0 velocity=2.0

Commit message: finish skrl transfer

File: assets/urdf/door_test/hook_test.urdf (robot description, URDF)
Before this commit: robot hook_test, 10 links, 9 joints
Links:
- added link hook_finger; visual sphere radius=0.007
Joints:
- added joint hook_finger: type fixed, parent hand_base, child hook_finger, origin xyz=0.08 0 0.17 rpy=0 0 0

Commit message: add door_handle spring and edit ur3 dof efforts

File: assets/urdf/door_test/hook_test.urdf (robot description, URDF)
Before this commit: robot hook_test, 11 links, 10 joints
Joints:
- joint ee_rx: limit lower=-0.1 upper=0.1 effort=10.0 velocity=2.0 -> lower=-0.1 upper=0.1 effort=10000.0 velocity=2.0
- joint ee_ry: limit lower=-0.1 upper=0.1 effort=10.0 velocity=2.0 -> lower=-0.1 upper=0.1 effort=10000.0 velocity=2.0
- joint ee_rz: limit lower=-0.1 upper=0.1 effort=10.0 velocity=2.0 -> lower=-0.1 upper=0.1 effort=10000.0 velocity=2.0
- joint ee_x: limit lower=-0.5 upper=1.0 effort=10.0 velocity=2.0 -> lower=-0.5 upper=1.0 effort=10000.0 velocity=2.0
- joint ee_y: limit lower=-0.2 upper=0.2 effort=10.0 velocity=2.0 -> lower=-0.2 upper=0.2 effort=10000.0 velocity=2.0
- joint ee_z: limit lower=-0.3 upper=0.3 effort=10.0 velocity=2.0 -> lower=-0.3 upper=0.3 effort=10000.0 velocity=2.0

Commit message: dof effort changed to open

File: assets/urdf/door_test/hook_test.urdf (robot description, URDF)
Before this commit: robot hook_test, 11 links, 10 joints
Joints:
- joint ee_rx: limit lower=-0.1 upper=0.1 effort=10000.0 velocity=2.0 -> lower=-0.1 upper=0.1 effort=100.0 velocity=2.0
- joint ee_ry: limit lower=-0.1 upper=0.1 effort=10000.0 velocity=2.0 -> lower=-0.1 upper=0.1 effort=100.0 velocity=2.0
- joint ee_rz: limit lower=-0.1 upper=0.1 effort=10000.0 velocity=2.0 -> lower=-0.1 upper=0.1 effort=100.0 velocity=2.0
- joint ee_x: limit lower=-0.5 upper=1.0 effort=10000.0 velocity=2.0 -> lower=-0.5 upper=1.0 effort=100.0 velocity=2.0
- joint ee_y: limit lower=-0.2 upper=0.2 effort=10000.0 velocity=2.0 -> lower=-0.2 upper=0.2 effort=100.0 velocity=2.0
- joint ee_z: limit lower=-0.3 upper=0.3 effort=10000.0 velocity=2.0 -> lower=-0.3 upper=0.3 effort=100.0 velocity=2.0

Commit message: change ur3 dof properties

File: assets/urdf/door_test/hook_test.urdf (robot description, URDF)
Before this commit: robot hook_test, 11 links, 10 joints
Joints:
- joint ee_rx: limit lower=-0.1 upper=0.1 effort=100.0 velocity=2.0 -> lower=-0.1 upper=0.1 effort=10.0 velocity=2.0
- joint ee_ry: limit lower=-0.1 upper=0.1 effort=100.0 velocity=2.0 -> lower=-0.1 upper=0.1 effort=10.0 velocity=2.0
- joint ee_rz: limit lower=-0.1 upper=0.1 effort=100.0 velocity=2.0 -> lower=-0.1 upper=0.1 effort=10.0 velocity=2.0
- joint ee_x: limit lower=-0.5 upper=1.0 effort=100.0 velocity=2.0 -> lower=-0.5 upper=1.0 effort=500.0 velocity=2.0
- joint ee_y: limit lower=-0.2 upper=0.2 effort=100.0 velocity=2.0 -> lower=-0.2 upper=0.2 effort=500.0 velocity=2.0
- joint ee_z: limit lower=-0.3 upper=0.3 effort=100.0 velocity=2.0 -> lower=-0.3 upper=0.3 effort=500.0 velocity=2.0

Commit message: reduce ur3 effort fuctor

File: assets/urdf/door_test/hook_test.urdf (robot description, URDF)
Before this commit: robot hook_test, 11 links, 10 joints
Joints:
- joint ee_x: limit lower=-0.5 upper=1.0 effort=500.0 velocity=2.0 -> lower=-0.5 upper=1.0 effort=100.0 velocity=2.0
- joint ee_y: limit lower=-0.2 upper=0.2 effort=500.0 velocity=2.0 -> lower=-0.2 upper=0.2 effort=100.0 velocity=2.0
- joint ee_z: limit lower=-0.3 upper=0.3 effort=500.0 velocity=2.0 -> lower=-0.3 upper=0.3 effort=100.0 velocity=2.0

Commit message: edit dof props

File: assets/urdf/door_test/hook_test.urdf (robot description, URDF)
Before this commit: robot hook_test, 11 links, 10 joints
Joints:
- joint ee_rx: limit lower=-1.0 upper=1.0 effort=10.0 velocity=2.0 -> lower=-1.0 upper=1.0 effort=10.0 velocity=5.0
- joint ee_ry: limit lower=-1.0 upper=1.0 effort=10.0 velocity=2.0 -> lower=-1.0 upper=1.0 effort=10.0 velocity=5.0
- joint ee_rz: limit lower=-1.0 upper=1.0 effort=10.0 velocity=2.0 -> lower=-1.0 upper=1.0 effort=10.0 velocity=5.0
- joint ee_x: limit lower=-1.0 upper=1.0 effort=100.0 velocity=2.0 -> lower=-1.0 upper=1.0 effort=100.0 velocity=5.0
- joint ee_y: limit lower=-1.0 upper=1.0 effort=100.0 velocity=2.0 -> lower=-1.0 upper=1.0 effort=100.0 velocity=5.0
- joint ee_z: limit lower=-1.0 upper=1.0 effort=100.0 velocity=2.0 -> lower=-1.0 upper=1.0 effort=100.0 velocity=5.0

Commit message: add non_vel

File: assets/urdf/door_test/hook_test.urdf (robot description, URDF)
Before this commit: robot hook_test, 11 links, 10 joints
Joints:
- joint ee_rx: limit lower=-1.0 upper=1.0 effort=10.0 velocity=5.0 -> lower=-1.0 upper=1.0 effort=10.0 velocity=5
- joint ee_ry: limit lower=-1.0 upper=1.0 effort=10.0 velocity=5.0 -> lower=-1.0 upper=1.0 effort=10.0 velocity=5
- joint ee_rz: limit lower=-1.0 upper=1.0 effort=10.0 velocity=5.0 -> lower=-1.0 upper=1.0 effort=10.0 velocity=5
- joint ee_x: limit lower=-1.0 upper=1.0 effort=100.0 velocity=5.0 -> lower=-1.0 upper=1.0 effort=100.0 velocity=5
- joint ee_y: limit lower=-1.0 upper=1.0 effort=100.0 velocity=5.0 -> lower=-1.0 upper=1.0 effort=100.0 velocity=5
- joint ee_z: limit lower=-1.0 upper=1.0 effort=100.0 velocity=5.0 -> lower=-1.0 upper=1.0 effort=100.0 velocity=5

Commit message: add EE from sagano_san

File: assets/urdf/door_test/hook_test.urdf (robot description, URDF)
Before this commit: robot hook_test, 11 links, 10 joints
Links:
- link hand_base: geometry collision cylinder length=0.065 radius=0.031; visual cylinder length=0.065 radius=0.02
- link hook: geometry collision mesh filename=./meshes/ur3/visual/hook4door_v3.obj; visual mesh filename=./meshes/ur3/visual/hook4door_sagano_san.dae scale=0.001 0.001 0.001
