Commit message: new doors added

File: assets/urdf/door_test/door_1_inv_wall_2.urdf (robot description, URDF)
Before this commit: robot door_test, 5 links, 4 joints
Links:
- link door_latch: geometry collision box size=0.001 0.5 0.01
Joints:
- joint base_joint: origin xyz=0 -0.5 0.0 rpy=0 0 0 -> xyz=0 0.5 0.0 rpy=0 0 3.14159
- joint door_handle: axis -1 0 0 -> 1 0 0
- joint door_hinge: axis 0 0 1 -> 0 0 -1; origin xyz=-0.07 0.972 0 rpy=3.14159 0 0 -> xyz=-0.07 0.06858 2.040

File: assets/urdf/door_test/door_2_inv_wall_2.urdf (robot description, URDF)
Before this commit: robot door_test, 5 links, 4 joints
Links:
- link door_latch: geometry collision box size=0.001 0.5 0.01
Joints:
- joint door_handle: origin xyz=0.035 0.75 -1.02 -> xyz=0.035 0.75 -1.0
- joint door_hinge: axis 0 0 1 -> 0 0 -1; limit lower=0 upper=1.57 effort=10000 velocity=100.00 -> lower=0 upper=1.57 effort=100 velocity=100.00; origin xyz=-0.07 0.972 0 rpy=3.14159 0 0 -> xyz=0.025 0.06858 0 rpy=0 3.14159 0

File: assets/urdf/door_test/hook_test.urdf (robot description, URDF)
Before this commit: robot hook_test, 11 links, 10 joints
Joints:
- joint ee_rx: limit lower=-1.0 upper=1.0 effort=10.0 velocity=5 -> lower=-1.0 upper=1.0 effort=10.0 velocity=5.0
- joint ee_ry: limit lower=-1.0 upper=1.0 effort=10.0 velocity=5 -> lower=-1.0 upper=1.0 effort=10.0 velocity=5.0
- joint ee_rz: limit lower=-1.0 upper=1.0 effort=10.0 velocity=5 -> lower=-1.0 upper=1.0 effort=10.0 velocity=5.0
- joint ee_x: limit lower=-1.0 upper=1.0 effort=100.0 velocity=5 -> lower=-1.0 upper=1.0 effort=100.0 velocity=5.0
- joint ee_y: limit lower=-1.0 upper=1.0 effort=100.0 velocity=5 -> lower=-1.0 upper=1.0 effort=100.0 velocity=5.0
- joint ee_z: limit lower=-1.0 upper=1.0 effort=100.0 velocity=5 -> lower=-1.0 upper=1.0 effort=100.0 velocity=5.0

Commit message: door urdf fidxed and started training

File: assets/urdf/door_test/door_1_inv_wall_2.urdf (robot description, URDF)
Before this commit: robot door_test, 5 links, 4 joints
Links:
- link door_handles: geometry collision mesh filename=./meshes/door_handle_collision.dae scale=1.23 1.27 0.7; collision mesh filename=./meshes/door_handle_collision.dae scale=1.23 1.27 0.7

File: assets/urdf/door_test/door_2_inv_wall_2.urdf (robot description, URDF)
Before this commit: robot door_test, 5 links, 4 joints
Links:
- link door_handles: geometry collision mesh filename=./meshes/door_handle_collision.dae scale=1.23 1.27 0.7; collision mesh filename=./meshes/door_handle_collision.dae scale=1.23 1.27 0.7

File: assets/urdf/door_test/door_2_wall.urdf (robot description, URDF)
Before this commit: robot door_test, 5 links, 4 joints
Links:
- link door_handles: geometry collision mesh filename=./meshes/door_handle_collision.dae scale=1.23 1.27 0.7; collision mesh filename=./meshes/door_handle_collision.dae scale=1.23 1.27 0.7
