Commit message: franka movie done

File: assets/urdf/door_test/v2_door_left_1.urdf (robot description, URDF)
Before this commit: robot door_test, 5 links, 4 joints
Links:
- link door: geometry collision mesh filename=./meshes/door.dae; visual mesh filename=./meshes/door.dae
- link door_handles: geometry collision mesh filename=./meshes/DH.stl scale=1.25 1.25 1.25; visual mesh filename=./meshes/DH-02201.dae scale=1.5 1.5 1.5
