Commit message: 座標系，ロボットのベー図座標系基準になっている

File: assets/urdf/door_test/hook_test_2.urdf (robot description, URDF)
Before this commit: robot hook_test, 11 links, 10 joints
Joints:
- joint ee_ry: parent ee_z_link -> ee_rx_link
- joint ee_rz: parent ee_z_link -> ee_ry_link

Commit message: 0702 done

File: assets/urdf/door_test/hook_test_2.urdf (robot description, URDF)
Before this commit: robot hook_test, 11 links, 10 joints
Joints:
- joint ee2hand_joint: parent ee_rz_link -> ee_rx_link
- joint ee_rx: parent ee_z_link -> ee_ry_link
- joint ee_ry: parent ee_rx_link -> ee_rz_link
- joint ee_rz: parent ee_ry_link -> ee_z_link

Commit message: while checking joint_space

File: assets/urdf/door_test/hook_test_2.urdf (robot description, URDF)
Before this commit: robot hook_test, 11 links, 10 joints
Joints:
- joint ee_rx: limit lower=-1.0 upper=1.0 effort=10.0 velocity=5.0 -> lower=-1.0 upper=1.0 effort=10.0 velocity=0.1
- joint ee_ry: limit lower=-1.0 upper=1.0 effort=10.0 velocity=5.0 -> lower=-1.0 upper=1.0 effort=10.0 velocity=0.1
- joint ee_rz: limit lower=-1.0 upper=1.0 effort=10.0 velocity=5.0 -> lower=-1.0 upper=1.0 effort=10.0 velocity=0.1
- joint ee_x: limit lower=-1.0 upper=1.0 effort=100.0 velocity=5.0 -> lower=-1.0 upper=1.0 effort=100.0 velocity=0.1
- joint ee_y: limit lower=-1.0 upper=1.0 effort=100.0 velocity=5.0 -> lower=-1.0 upper=1.0 effort=100.0 velocity=0.1
- joint ee_z: limit lower=-1.0 upper=1.0 effort=100.0 velocity=5.0 -> lower=-1.0 upper=1.0 effort=100.0 velocity=0.1
