Commit message: add robot_helper, while adding transforming action

File: assets/urdf/door_test/v2_hook_hand.urdf (robot description, URDF)
Before this commit: robot hook_hand, 10 links, 9 joints
Joints:
- joint ee_rx: limit lower=-1.0 upper=1.0 effort=10.0 velocity=0.1 -> lower=-3.1415926 upper=3.1415926 effort=100.0 velocity=0.1
- joint ee_ry: limit lower=-1.0 upper=1.0 effort=10.0 velocity=0.1 -> lower=-3.1415926 upper=3.1415926 effort=100.0 velocity=0.1
- joint ee_rz: limit lower=-1.0 upper=1.0 effort=10.0 velocity=0.1 -> lower=-3.1415926 upper=3.1415926 effort=100.0 velocity=0.1
- joint ee_x: limit lower=-1.0 upper=1.0 effort=100.0 velocity=0.1 -> lower=-2.0 upper=2.0 effort=100.0 velocity=0.1
- joint ee_y: limit lower=-1.0 upper=1.0 effort=100.0 velocity=0.1 -> lower=-2.0 upper=2.0 effort=100.0 velocity=0.1
- joint ee_z: limit lower=-1.0 upper=1.0 effort=100.0 velocity=0.1 -> lower=-2.0 upper=2.0 effort=100.0 velocity=0.1

Commit message: adding pixel missing, while transformation

File: assets/urdf/door_test/v2_hook_hand.urdf (robot description, URDF)
Before this commit: robot hook_hand, 10 links, 9 joints
Joints:
- joint ee_rx: limit lower=-3.1415926 upper=3.1415926 effort=100.0 velocity=0.1 -> lower=-6.28 upper=6.28 effort=100.0 velocity=0.1
- joint ee_ry: limit lower=-3.1415926 upper=3.1415926 effort=100.0 velocity=0.1 -> lower=-6.28 upper=6.28 effort=100.0 velocity=0.1
- joint ee_rz: limit lower=-3.1415926 upper=3.1415926 effort=100.0 velocity=0.1 -> lower=-6.28 upper=6.28 effort=100.0 velocity=0.1

Commit message: edit hook_finger pose

File: assets/urdf/door_test/v2_hook_hand.urdf (robot description, URDF)
Before this commit: robot hook_hand, 10 links, 9 joints
Joints:
- joint hook_finger: origin xyz=0.08 0 0.17 rpy=0 0 0 -> xyz=0.08 0 0.17 rpy=0 -1.57 0
