Commit message: handle size changed

File: assets/urdf/door_test/door_1_inv_wall.urdf (robot description, URDF)
Before this commit: robot door_test, 5 links, 4 joints
Links:
- link door_handles: geometry collision mesh filename=./meshes/door_handle.dae scale=1.0 0.75 0.75; collision mesh filename=./meshes/door_handle.dae scale=1.0 0.75 0.75

File: assets/urdf/door_test/door_1_wall.urdf (robot description, URDF)
Before this commit: robot door_test, 5 links, 4 joints
Links:
- link door_handles: geometry collision mesh filename=./meshes/door_handle.dae scale=1.0 0.75 0.75; collision mesh filename=./meshes/door_handle.dae scale=1.0 0.75 0.75

File: assets/urdf/door_test/door_2_inv_wall.urdf (robot description, URDF)
Before this commit: robot door_test, 5 links, 4 joints
Links:
- link door_handles: geometry collision mesh filename=./meshes/door_handle.dae scale=1.0 0.75 0.75; collision mesh filename=./meshes/door_handle.dae scale=1.0 0.75 0.75

File: assets/urdf/door_test/door_2_wall.urdf (robot description, URDF)
Before this commit: robot door_test, 5 links, 4 joints
Links:
- link door_handles: geometry collision mesh filename=./meshes/door_handle.dae scale=1.0 0.75 0.75; collision mesh filename=./meshes/door_handle.dae scale=1.0 0.75 0.75

Commit message: fix door_handle urdf bug

File: assets/urdf/door_test/door_1_inv_wall.urdf (robot description, URDF)
Before this commit: robot door_test, 5 links, 4 joints
Links:
- link door_handles: geometry collision mesh filename=./meshes/door_handle_collision.dae scale=1.0 0.75 0.75; collision mesh filename=./meshes/door_handle_collision.dae scale=1.0 0.75 0.75

File: assets/urdf/door_test/door_1_wall.urdf (robot description, URDF)
Before this commit: robot door_test, 5 links, 4 joints
Links:
- link door_handles: geometry collision mesh filename=./meshes/door_handle_collision.dae scale=1.0 0.75 0.75; collision mesh filename=./meshes/door_handle_collision.dae scale=1.0 0.75 0.75

File: assets/urdf/door_test/door_2_inv_wall.urdf (robot description, URDF)
Before this commit: robot door_test, 5 links, 4 joints
Links:
- link door_handles: geometry collision mesh filename=./meshes/door_handle_collision.dae scale=1.0 0.75 0.75; collision mesh filename=./meshes/door_handle_collision.dae scale=1.0 0.75 0.75

File: assets/urdf/door_test/door_2_wall.urdf (robot description, URDF)
Before this commit: robot door_test, 5 links, 4 joints
Links:
- link door_handles: geometry collision mesh filename=./meshes/door_handle_collision.dae scale=1.0 0.75 0.75; collision mesh filename=./meshes/door_handle_collision.dae scale=1.0 0.75 0.75

Commit message: change all door handle to shirokuma

File: assets/urdf/door_test/door_1_inv_wall.urdf (robot description, URDF)
Before this commit: robot door_test, 5 links, 4 joints
Links:
- link door_handles: geometry collision mesh filename=./meshes/shirokuma_scaled_collision.stl; collision mesh filename=./meshes/shirokuma_scaled_collision.stl
Joints:
- joint base_joint: origin xyz=0 -0.5 0.0 rpy=0 0 0 -> xyz=0 0.5 0.0 rpy=0 0 3.14159
- joint door_handle: axis -1 0 0 -> 1 0 0; origin xyz=0.035 0.75 -1.0 -> xyz=0.035 0.75 -1.02
- joint door_hinge: limit lower=0 upper=1.57 effort=100 velocity=100.00 -> lower=0 upper=1.57 effort=10000 velocity=100.00; origin xyz=0.025 0.06858 0 rpy=0 3.14159 0 -> xyz=-0.07 0.06858 2.040

File: assets/urdf/door_test/door_2_inv_wall.urdf (robot description, URDF)
Before this commit: robot door_test, 5 links, 4 joints
Links:
- link door_handles: geometry collision mesh filename=./meshes/shirokuma_scaled_collision.stl; collision mesh filename=./meshes/shirokuma_scaled_collision.stl
- link door_latch: geometry collision box size=0.001 0.5 0.01
Joints:
- joint base_joint: origin xyz=0 0.5 0.0 rpy=0 0 3.14159 -> xyz=0 -0.5 0.0 rpy=0 0 0
- joint door_handle: axis 1 0 0 -> -1 0 0; origin xyz=0.035 0.75 -1.02 -> xyz=0.035 0.75 -1.0
- joint door_hinge: axis 0 0 1 -> 0 0 -1; limit lower=0 upper=1.57 effort=10000 velocity=100.00 -> lower=0 upper=1.57 effort=100 velocity=100.00; origin xyz=-0.07 0.06858 2.040 -> xyz=0.025 0.06858 0 rpy=0 3.14159 0

File: assets/urdf/door_test/door_2_wall.urdf (robot description, URDF)
Before this commit: robot door_test, 5 links, 4 joints
Links:
- link door_handles: geometry collision mesh filename=./meshes/shirokuma_scaled_collision.stl; collision mesh filename=./meshes/shirokuma_scaled_collision.stl
Joints:
- joint door_handle: origin xyz=0.035 0.75 -1.0 -> xyz=0.035 0.75 -1.02

Commit message: start learning

File: assets/urdf/door_test/door_1_inv_wall.urdf (robot description, URDF)
Before this commit: robot door_test, 5 links, 4 joints
Links:
- added link door_fake_link
Joints:
- added joint base_to_door_fake_link: type fixed, parent base_link, child door_fake_link, origin xyz=0.5 0 0.0 rpy=0 0 3.14159

File: assets/urdf/door_test/door_1_wall.urdf (robot description, URDF)
Before this commit: robot door_test, 5 links, 4 joints
Links:
- added link door_fake_link
Joints:
- added joint base_to_door_fake_link: type fixed, parent base_link, child door_fake_link, origin xyz=0.5 0 0.0 rpy=0 0 3.14159

File: assets/urdf/door_test/door_2_inv_wall.urdf (robot description, URDF)
Before this commit: robot door_test, 5 links, 4 joints
Links:
- added link door_fake_link
Joints:
- added joint base_to_door_fake_link: type fixed, parent base_link, child door_fake_link, origin xyz=0.5 0 0.0 rpy=0 0 3.14159

File: assets/urdf/door_test/door_2_wall.urdf (robot description, URDF)
Before this commit: robot door_test, 5 links, 4 joints
Links:
- added link door_fake_link
Joints:
- added joint base_to_door_fake_link: type fixed, parent base_link, child door_fake_link, origin xyz=0.5 0 0.0 rpy=0 0 3.14159

Commit message: add hook_finger dsr_pose

File: assets/urdf/door_test/door_1_inv_wall.urdf (robot description, URDF)
Before this commit: robot door_test, 6 links, 5 joints
Links:
- added link dsr_pose
Joints:
- added joint handle2dsr_pose: type fixed, parent door_handles, child dsr_pose, origin xyz=-0.07 -0.13 -0.05

File: assets/urdf/door_test/door_1_wall.urdf (robot description, URDF)
Before this commit: robot door_1_wall, 6 links, 5 joints
Links:
- added link dsr_pose
Joints:
- added joint handle2dsr_pose: type fixed, parent door_handles, child dsr_pose, origin xyz=-0.07 -0.13 -0.05

File: assets/urdf/door_test/door_2_inv_wall.urdf (robot description, URDF)
Before this commit: robot door_test, 6 links, 5 joints
Links:
- added link dsr_pose
Joints:
- added joint handle2dsr_pose: type fixed, parent door_handles, child dsr_pose, origin xyz=-0.07 -0.13 0.05 rpy=3.14159265 0 0

File: assets/urdf/door_test/door_2_wall.urdf (robot description, URDF)
Before this commit: robot door_test, 6 links, 5 joints
Links:
- added link dsr_pose
Joints:
- added joint handle2dsr_pose: type fixed, parent door_handles, child dsr_pose, origin xyz=-0.07 -0.13 0.05 rpy=3.14159265 0 0

Commit message: fix dsr_pose rotations

File: assets/urdf/door_test/door_1_inv_wall.urdf (robot description, URDF)
Before this commit: robot door_test, 7 links, 6 joints
Joints:
- joint handle2dsr_pose: origin xyz=-0.07 -0.13 -0.05 -> xyz=-0.07 -0.13 -0.05 rpy=0 0 3.14159265

File: assets/urdf/door_test/door_1_wall.urdf (robot description, URDF)
Before this commit: robot door_1_wall, 7 links, 6 joints
Joints:
- joint handle2dsr_pose: origin xyz=-0.07 -0.13 -0.05 -> xyz=-0.07 -0.13 -0.05 rpy=0 0 3.14159265

File: assets/urdf/door_test/door_2_inv_wall.urdf (robot description, URDF)
Before this commit: robot door_test, 7 links, 6 joints
Joints:
- joint handle2dsr_pose: origin xyz=-0.07 -0.13 0.05 rpy=3.14159265 0 0 -> xyz=-0.07 -0.13 0.05 rpy=3.14159265 0 3.14159265

File: assets/urdf/door_test/door_2_wall.urdf (robot description, URDF)
Before this commit: robot door_test, 7 links, 6 joints
Joints:
- joint handle2dsr_pose: origin xyz=-0.07 -0.13 0.05 rpy=3.14159265 0 0 -> xyz=-0.07 -0.13 0.05 rpy=3.14159265 0 3.14159265

Commit message: move dsr_pose

File: assets/urdf/door_test/door_1_inv_wall.urdf (robot description, URDF)
Before this commit: robot door_test, 7 links, 6 joints
Joints:
- joint handle2dsr_pose: origin xyz=-0.07 -0.13 -0.05 rpy=0 0 3.14159265 -> xyz=-0.03 -0.13 0.0 rpy=0 0 3.14159265

File: assets/urdf/door_test/door_1_wall.urdf (robot description, URDF)
Before this commit: robot door_1_wall, 7 links, 6 joints
Joints:
- joint handle2dsr_pose: origin xyz=-0.07 -0.13 -0.05 rpy=0 0 3.14159265 -> xyz=-0.03 -0.13 0.0 rpy=0 0 3.14159265

File: assets/urdf/door_test/door_2_inv_wall.urdf (robot description, URDF)
Before this commit: robot door_test, 7 links, 6 joints
Joints:
- joint handle2dsr_pose: origin xyz=-0.07 -0.13 0.05 rpy=3.14159265 0 3.14159265 -> xyz=-0.03 -0.13 0.0 rpy=3.14159265 0 3.14159265

File: assets/urdf/door_test/door_2_wall.urdf (robot description, URDF)
Before this commit: robot door_test, 7 links, 6 joints
Joints:
- joint handle2dsr_pose: origin xyz=-0.07 -0.13 0.05 rpy=3.14159265 0 3.14159265 -> xyz=-0.03 -0.13 0.0 rpy=3.14159265 0 3.14159265

Commit message: change door_latch origin into joint

File: assets/urdf/door_test/door_1_inv_wall.urdf (robot description, URDF)
Before this commit: robot door_test, 7 links, 6 joints
Joints:
- joint handle2latch: origin (none) -> xyz=-0.014 0.2 0.9 rpy=0 0 0

File: assets/urdf/door_test/door_1_wall.urdf (robot description, URDF)
Before this commit: robot door_1_wall, 7 links, 6 joints
Joints:
- joint handle2latch: origin (none) -> xyz=0.043 0.1 0 rpy=0 0 0

File: assets/urdf/door_test/door_2_wall.urdf (robot description, URDF)
Before this commit: robot door_test, 7 links, 6 joints
Joints:
- joint handle2latch: origin (none) -> xyz=0.043 0.1 0 rpy=0 0 0
