Commit message: fix door inv urdrs

File: assets/urdf/door_test/door_2_inv_wall.urdf (robot description, URDF)
Before this commit: robot door_test, 5 links, 4 joints
Links:
- link door_latch: geometry collision box size=0.001 0.13 0.01

Commit message: fix door_2_inv_wall bug

File: assets/urdf/door_test/door_2_inv_wall.urdf (robot description, URDF)
Before this commit: robot door_test, 7 links, 6 joints
Joints:
- joint handle2latch: origin (none) -> xyz=-0.018 0.2 -0.9 rpy=0 0 0

Commit message: edit door_2_inv_wall.urdf : enlarge wall size

File: assets/urdf/door_test/door_2_inv_wall.urdf (robot description, URDF)
Before this commit: robot door_test, 7 links, 6 joints
Links:
- link door_wall: geometry collision box size=0.05029 0.06858 2.10820; collision box size=0.08 2.0 3.0

File: assets/urdf/door_test/door_2_wall.urdf (robot description, URDF)
Before this commit: robot door_test, 7 links, 6 joints
Links:
- link door_wall: geometry collision box size=0.05029 0.06858 2.10820; collision box size=0.08 2.0 3.0
