Commit message: edit door scales

File: assets/urdf/door_test/prev_door_1_inv_wall.urdf (robot description, URDF)
Before this commit: robot door_test, 5 links, 4 joints
Links:
- link door_handles: geometry collision mesh filename=./meshes/door_handle_collision.dae; collision mesh filename=./meshes/door_handle_collision.dae

File: assets/urdf/door_test/prev_door_1_wall.urdf (robot description, URDF)
Before this commit: robot door_test, 5 links, 4 joints
Links:
- link door_handles: geometry collision mesh filename=./meshes/door_handle_collision.dae; collision mesh filename=./meshes/door_handle_collision.dae

File: assets/urdf/door_test/prev_door_2_inv_wall.urdf (robot description, URDF)
Before this commit: robot door_test, 5 links, 4 joints
Links:
- link door_handles: geometry collision mesh filename=./meshes/door_handle_collision.dae; collision mesh filename=./meshes/door_handle_collision.dae

File: assets/urdf/door_test/prev_door_2_wall.urdf (robot description, URDF)
Before this commit: robot door_test, 5 links, 4 joints
Links:
- link door_handles: geometry collision mesh filename=./meshes/door_handle_collision.dae; collision mesh filename=./meshes/door_handle_collision.dae

Commit message: add dsr_poses into urdfs

File: assets/urdf/door_test/prev_door_1_inv_wall.urdf (robot description, URDF)
Before this commit: robot door_test, 5 links, 4 joints
Links:
- added link dsr_pose
Joints:
- added joint handle2dsr_pose: type fixed, parent door_handles, child dsr_pose, origin xyz=-0.07 -0.13 -0.02

File: assets/urdf/door_test/prev_door_1_wall.urdf (robot description, URDF)
Before this commit: robot door_test, 5 links, 4 joints
Links:
- added link dsr_pose
Joints:
- added joint handle2dsr_pose: type fixed, parent door_handles, child dsr_pose, origin xyz=-0.07 -0.13 -0.02

File: assets/urdf/door_test/prev_door_2_inv_wall.urdf (robot description, URDF)
Before this commit: robot door_test, 5 links, 4 joints
Links:
- added link dsr_pose
Joints:
- added joint handle2dsr_pose: type fixed, parent door_handles, child dsr_pose, origin xyz=-0.07 -0.13 0.02 rpy=3.14159265 0 0

File: assets/urdf/door_test/prev_door_2_wall.urdf (robot description, URDF)
Before this commit: robot door_test, 5 links, 4 joints
Links:
- added link dsr_pose
Joints:
- added joint handle2dsr_pose: type fixed, parent door_handles, child dsr_pose, origin xyz=-0.07 -0.13 0.02 rpy=3.14159265 0 0

Commit message: add modified prev_door urdfs

File: assets/urdf/door_test/prev_door_1_inv_wall.urdf (robot description, URDF)
Before this commit: robot door_test, 7 links, 6 joints
Links:
- link door_handles: geometry collision mesh filename=./meshes/door_handle_collision.dae; collision mesh filename=./meshes/door_handle_collision.dae
Joints:
- joint base_joint: origin xyz=0 -0.5 0.0 rpy=0 0 0 -> xyz=0 0.5 0.0 rpy=0 0 3.14159
- joint door_handle: axis -1 0 0 -> 1 0 0; origin xyz=0.035 0.75 -1.0 -> xyz=0.035 0.75 -1.02
- joint door_hinge: limit lower=0 upper=1.57 effort=100 velocity=100.00 -> lower=0 upper=1.57 effort=10000 velocity=100.00; origin xyz=0.025 0.06858 0 rpy=0 3.14159 0 -> xyz=-0.07 0.06858 2.040
- joint handle2dsr_pose: origin xyz=-0.03 -0.13 0.0 rpy=3.14159265 0 3.14159265 -> xyz=-0.03 -0.13 0.0 rpy=0 0 3.14159265
- joint handle2latch: origin xyz=-0.018 0.2 -0.9 rpy=0 0 0 -> (none)

File: assets/urdf/door_test/prev_door_1_wall.urdf (robot description, URDF)
Before this commit: robot door_test, 7 links, 6 joints
Links:
- link door_handles: geometry collision mesh filename=./meshes/door_handle_collision.dae; collision mesh filename=./meshes/door_handle_collision.dae
- link door_latch: geometry collision box size=0.001 0.14 0.01
Joints:
- joint base_joint: origin xyz=0 -0.5 0.0 rpy=0 0 0 -> xyz=0 0.5 0.0 rpy=0 0 3.14159
- joint door_handle: axis -1 0 0 -> 1 0 0; origin xyz=0.035 0.75 -1.0 -> xyz=0.035 0.75 -1.02
- joint door_hinge: axis 0 0 -1 -> 0 0 1; limit lower=0 upper=1.57 effort=100 velocity=100.00 -> lower=0 upper=1.57 effort=10000 velocity=100.00; origin xyz=0.025 0.06858 0 rpy=0 3.14159 0 -> xyz=-0.07 0.06858 2.040
- joint handle2dsr_pose: origin xyz=-0.03 -0.13 0.0 rpy=3.14159265 0 3.14159265 -> xyz=-0.03 -0.13 0.0 rpy=0 0 3.14159265
- joint handle2latch: origin xyz=-0.018 0.2 -0.9 rpy=0 0 0 -> (none)

File: assets/urdf/door_test/prev_door_2_inv_wall.urdf (robot description, URDF)
Before this commit: robot door_test, 7 links, 6 joints
Links:
- link door_handles: geometry collision mesh filename=./meshes/door_handle_collision.dae; collision mesh filename=./meshes/door_handle_collision.dae
Joints:
- joint handle2latch: origin xyz=-0.018 0.2 -0.9 rpy=0 0 0 -> (none)

File: assets/urdf/door_test/prev_door_2_wall.urdf (robot description, URDF)
Before this commit: robot door_test, 7 links, 6 joints
Links:
- link door_handles: geometry collision mesh filename=./meshes/door_handle_collision.dae; collision mesh filename=./meshes/door_handle_collision.dae
- link door_latch: geometry collision box size=0.001 0.14 0.01
Joints:
- joint door_hinge: axis 0 0 -1 -> 0 0 1
- joint handle2latch: origin xyz=-0.018 0.2 -0.9 rpy=0 0 0 -> (none)

Commit message: change dsr_pose and dist_thresh

File: assets/urdf/door_test/prev_door_1_inv_wall.urdf (robot description, URDF)
Before this commit: robot door_test, 7 links, 6 joints
Joints:
- joint handle2dsr_pose: origin xyz=-0.03 -0.13 0.0 rpy=0 0 3.14159265 -> xyz=-0.03 -0.11 0.0 rpy=0 0 3.14159265

File: assets/urdf/door_test/prev_door_1_wall.urdf (robot description, URDF)
Before this commit: robot door_test, 7 links, 6 joints
Joints:
- joint handle2dsr_pose: origin xyz=-0.03 -0.13 0.0 rpy=0 0 3.14159265 -> xyz=-0.03 -0.11 0.0 rpy=0 0 3.14159265

File: assets/urdf/door_test/prev_door_2_inv_wall.urdf (robot description, URDF)
Before this commit: robot door_test, 7 links, 6 joints
Joints:
- joint handle2dsr_pose: origin xyz=-0.03 -0.13 0.0 rpy=3.14159265 0 3.14159265 -> xyz=-0.03 -0.11 0.0 rpy=3.14159265 0 3.14159265

File: assets/urdf/door_test/prev_door_2_wall.urdf (robot description, URDF)
Before this commit: robot door_test, 7 links, 6 joints
Joints:
- joint handle2dsr_pose: origin xyz=-0.03 -0.13 0.0 rpy=3.14159265 0 3.14159265 -> xyz=-0.03 -0.11 0.0 rpy=3.14159265 0 3.14159265
