Commit message: new branch sim2real

File: assets/urdf/door_test/door_1_wall.urdf (robot description, URDF)
Before this commit: robot door_test, 5 links, 4 joints
Links:
- link door_handles: geometry collision mesh filename=./meshes/door_handle_collision.dae scale=1.23 1.27 0.7; collision mesh filename=./meshes/door_handle_collision.dae scale=1.23 1.27 0.7

Commit message: edit door_1_wall.urdf : enlarge wall

File: assets/urdf/door_test/door_1_wall.urdf (robot description, URDF)
Before this commit: robot door_1_wall, 7 links, 6 joints
Links:
- link door_wall: geometry collision box size=0.05029 0.06858 2.10820; collision box size=0.08 2.0 3.0

Commit message: edit dsr_pose of pull doors

File: assets/urdf/door_test/door_1_wall.urdf (robot description, URDF)
Before this commit: robot door_1_wall, 7 links, 6 joints
Joints:
- joint handle2dsr_pose: origin xyz=-0.03 -0.13 0.0 rpy=0 0 3.14159265 -> xyz=-0.03 -0.13 0.0 rpy=0 0.2617 3.14159265

File: assets/urdf/door_test/door_2_wall.urdf (robot description, URDF)
Before this commit: robot door_test, 7 links, 6 joints
Joints:
- joint handle2dsr_pose: origin xyz=-0.03 -0.13 0.0 rpy=3.14159265 0 3.14159265 -> xyz=-0.03 -0.13 0.0 rpy=3.14159265 -0.2617 3.14159265

File: assets/urdf/door_test/prev_door_1_wall.urdf (robot description, URDF)
Before this commit: robot door_test, 7 links, 6 joints
Joints:
- joint handle2dsr_pose: origin xyz=-0.03 -0.11 0.0 rpy=0 0 3.14159265 -> xyz=-0.03 -0.11 0.0 rpy=0 0.2617 3.14159265

File: assets/urdf/door_test/prev_door_2_wall.urdf (robot description, URDF)
Before this commit: robot door_test, 7 links, 6 joints
Joints:
- joint handle2dsr_pose: origin xyz=-0.03 -0.11 0.0 rpy=3.14159265 0 3.14159265 -> xyz=-0.03 -0.11 0.0 rpy=3.14159265 -0.2617 3.14159265
