Commit message: add left hinge door into door_hook.py

File: assets/urdf/kuka_allegro_description/door_2.urdf (robot description, URDF)
Before this commit: robot door_test, 5 links, 4 joints
Joints:
- joint base_joint: origin xyz=0 -0.5 0.0 rpy=0 0 0 -> xyz=0 0.5 0.0 rpy=0 0 0
- joint door_hinge: origin xyz=0.025 0.06858 0 rpy=0 3.14159 0 -> xyz=0.525 0.06858 0 rpy=0 3.14159 0
