Commit message: minor changes

File: assets/urdf/franka_description/robots/franka_hook.urdf (robot description, URDF)
Before this commit: robot panda, 12 links, 11 joints
Links:
- link hook: geometry collision mesh filename=./meshes/ur3/visual/hook4door_v3.obj; visual mesh filename=./meshes/ur3/visual/hook4door_sagano_san.dae scale=0.001 0.001 0.001
